File: Ergogen/output/pcbs/ergogen_pcb_tutorial.kicad_pcb (KiCad board)
At the start: 2 copper layers, 237.3 x 104.4 mm, 73 parts

Commit message: updating ergogen layout
Parts:
- added JST1: , JST_PH_S2B-PH-K_02x2.00mm_Angled, F.Cu at (172.0, 145.7)
- added T1: , E73:SPDT_C128955, F.Cu at (172.0, 155.2)
- MCU1: value (none) -> nice_nano; footprint ProMicro -> nice_nano
- moved MCU1 4.75 mm to (172.0, 126.7)
- moved D12 4.50 mm to (131.1, 106.3)
- moved D13 4.50 mm to (137.8, 148.3)
- moved D14 4.50 mm to (143.5, 130.2)
- moved D15 4.50 mm to (149.2, 112.1)
- moved D17 4.50 mm to (132.1, 166.4)
- moved D18 4.50 mm to (150.2, 172.1)
- moved D23 4.50 mm to (255.0, 113.0)
- moved D24 4.50 mm to (249.2, 94.9)
- moved D25 4.50 mm to (239.7, 127.8)
- moved D26 4.50 mm to (234.0, 109.7)
- moved D27 4.50 mm to (228.3, 91.6)
- moved D28 4.50 mm to (224.4, 142.6)
- moved D29 4.50 mm to (218.7, 124.5)
- moved D30 4.50 mm to (213.0, 106.3)
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Connections:
- net P1 renamed P009
- net P15 renamed P100
- net P18 renamed P024
- net P19 renamed P022
- net P20 renamed P020
- net P21 renamed P017
- D1 pad 1: P8 -> P104
- D10 pad 1: P8 -> P104
- D11 pad 1: P16 -> P010
- D12 pad 1: P14 -> P111
- D13 pad 1: P8 -> P104
- D14 pad 1: P16 -> P010
- D15 pad 1: P14 -> P111
- D16 pad 1: P9 -> P106
- D17 pad 1: P9 -> P106
- D18 pad 1: P9 -> P106
- D19 pad 1: P8 -> P104
- D2 pad 1: P16 -> P010
- D20 pad 1: P16 -> P010
- D21 pad 1: P14 -> P111
- D22 pad 1: P8 -> P104
- D23 pad 1: P16 -> P010
- D24 pad 1: P14 -> P111
- D25 pad 1: P8 -> P104
- D26 pad 1: P16 -> P010
- D27 pad 1: P14 -> P111
- D28 pad 1: P8 -> P104
- D29 pad 1: P16 -> P010
- D3 pad 1: P14 -> P111
- D30 pad 1: P14 -> P111
- D31 pad 1: P8 -> P104
- D32 pad 1: P16 -> P010
- D33 pad 1: P14 -> P111
- D34 pad 1: P9 -> P106
- D35 pad 1: P9 -> P106
- D36 pad 1: P9 -> P106
- D4 pad 1: P8 -> P104
- D5 pad 1: P16 -> P010
- D6 pad 1: P14 -> P111
- D7 pad 1: P8 -> P104
- D8 pad 1: P16 -> P010
- D9 pad 1: P14 -> P111
- MCU1 pad 1: RAW -> pos
- MCU1 pad 10: P14 -> P011
- MCU1 pad 11: P16 -> P104
- MCU1 pad 12: P10 -> P106
- MCU1 pad 14: P0 -> P010
- MCU1 pad 15: GND -> P111
- MCU1 pad 16: GND -> P113
- MCU1 pad 17: P2 -> P115
- MCU1 pad 18: P3 -> P002
- MCU1 pad 19: P4 -> P029
- MCU1 pad 2: GND -> P008
- MCU1 pad 20: P5 -> P031
- MCU1 pad 21: P6 -> VCC
- MCU1 pad 22: P7 -> RST
- MCU1 pad 23: P8 -> GND
- MCU1 pad 24: P9 -> RAW
- MCU1 pad 3: RST -> GND
- MCU1 pad 4: VCC -> GND
- S19 pad 1: P2 -> P031
- S20 pad 1: P2 -> P031
- S21 pad 1: P2 -> P031
- S22 pad 1: P3 -> P029
- S23 pad 1: P3 -> P029
- S24 pad 1: P3 -> P029
- S25 pad 1: P4 -> P002
- S26 pad 1: P4 -> P002
- S27 pad 1: P4 -> P002
- S28 pad 1: P5 -> P115
- S29 pad 1: P5 -> P115
- S30 pad 1: P5 -> P115
- S31 pad 1: P6 -> P113
- S32 pad 1: P6 -> P113
- S33 pad 1: P6 -> P113
- S34 pad 1: P4 -> P002
- S35 pad 1: P5 -> P115
- S36 pad 1: P6 -> P113
Other:
- board size 237.3 x 104.4 mm -> 242.3 x 109.4 mm

Commit message: more updates to ergogen config
Parts:
- T1: footprint E73:SPDT_C128955 -> josh_custom:1test slide switch
- moved T1 2.84 mm to (172.0, 152.4)
- turned S5 to -17 degrees
- turned S26 to 18 degrees
- turned S30 to 18 degrees
- turned D35 to 18 degrees
- turned D5 to -17 degrees
- turned D27 to 18 degrees
- turned D6 to -17 degrees
- turned S27 to 18 degrees
- turned D30 to 18 degrees
- turned D36 to 18 degrees
- turned S2 to -17 degrees
- turned S8 to -17 degrees
- turned S29 to 18 degrees
- turned D29 to 18 degrees
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Routing:
- net P111: track 0.00 -> 290.6 mm, vias 0 -> 5
- net P010: track 0.00 -> 282.4 mm, vias 0 -> 5
- net P104: track 0.00 -> 260.4 mm, vias 0 -> 2
- net P017: track 0.00 -> 151.2 mm, vias 0 -> 1
- net P002: track 0.00 -> 133.7 mm, vias 0 -> 1
- net P024: track 0.00 -> 132.7 mm, vias 0 -> 3
- net P031: track 0.00 -> 132.5 mm, vias 0 -> 1
- net P020: track 0.00 -> 128.7 mm, vias 0 -> 1
- net P029: track 0.00 -> 112.5 mm, vias 0 -> 1
- net P115: track 0.00 -> 105.7 mm
- net P100: track 0.00 -> 96.0 mm
- net P113: track 0.00 -> 82.9 mm, vias 0 -> 1
- net P022: track 0.00 -> 82.2 mm
- net P106: track 0.00 -> 65.0 mm
- net RAW: track 0.00 -> 41.7 mm
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- added copper zone on B.Cu, net (none)
- added copper zone on F.Cu, net (none)
Other:
- net class Default removed
