File: ergogenrp2040zero/output/pcbs/wired_pcb_ergo_wip.kicad_pcb (KiCad board)
At the start: 2 copper layers, 238.6 x 105.6 mm, 74 parts

Commit message: experimental jscad ergogen outputs for cases
Parts:
- removed G***: LOGO, custom graphics library:start trek test 2
- moved S13 17.1 mm to (140.6, 139.2)
- moved S14 17.1 mm to (146.4, 121.1)
- moved S21 17.1 mm to (267.4, 89.2)
- moved D5 17.1 mm to (89.4, 112.1)
- moved S15 17.1 mm to (152.1, 103.0)
- moved D27 17.1 mm to (228.0, 90.6)
- moved S30 17.1 mm to (210.1, 97.3)
- moved D30 17.1 mm to (212.7, 105.4)
- moved D32 17.1 mm to (200.3, 129.2)
- moved D4 17.1 mm to (83.7, 130.2)
- moved S19 17.1 mm to (278.8, 125.4)
- moved D12 17.1 mm to (131.4, 105.4)
- moved S25 17.1 mm to (236.8, 118.7)
- moved D15 17.1 mm to (149.5, 111.1)
- moved S18 17.1 mm to (153.0, 163.1)
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Routing:
- net P9: track 267.2 -> 0.00 mm
- net P8: track 245.6 -> 0.00 mm
- net P2: track 232.8 -> 0.00 mm
- net P27: track 199.4 -> 0.00 mm
- net P5: track 179.9 -> 0.00 mm
- net P29: track 172.8 -> 0.00 mm
- net P11: track 165.7 -> 0.00 mm
- net P3: track 165.3 -> 0.00 mm
- net P28: track 150.6 -> 0.00 mm
- net P26: track 149.6 -> 0.00 mm
- net P6: track 140.6 -> 0.00 mm
- net P4: track 138.2 -> 0.00 mm
- net P15: track 101.7 -> 0.00 mm
- net P7: track 76.4 -> 0.00 mm
- net middle_bottom: track 14.9 -> 0.00 mm
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- removed copper zone on B.Cu, net (none)
- removed copper zone on F.Cu, net (none)
Other:
- outline, holes or cut-outs redrawn
- net class Default added: clearance 0.2, trace_width 0.25, via_dia 0.8, via_drill 0.4
